File: RN4020_Breakout/RevA.brd (EAGLE design)
At the start: 25.5 x 30.5 mm, 3 parts

Commit message: Made artwork revisions to fit Itead manufacturing limitations
Connections:
- net N$12 renamed VDD
Other:
- board text added: "REV_A"
- board text removed: "REVA"
