File: RN4020_Breakout/RevA.sch (EAGLE design)
At the start: 3 parts

Commit message: Made artwork revisions to fit Itead manufacturing limitations
Connections:
- net N$12 renamed VDD
Changed lines of the file:
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@@
 <pinref part="JP1" gate="G$1" pin="1"/>
 <wire x1="-33.02" y1="20.32" x2="-68.58" y2="20.32" width="0.1524" layer="91"/>
+<label x="-66.04" y="20.32" size="1.778" layer="95"/>
 </segment>
 <segment>
@@
 <pinref part="JP2" gate="G$1" pin="1"/>
 <wire x1="33.02" y1="20.32" x2="68.58" y2="20.32" width="0.1524" layer="91"/>
+<label x="58.42" y="20.32" size="1.778" layer="95"/>
 </segment>
 </net>
@@
 </segment>
 </net>
-<net name="N$12" class="0">
+<net name="VDD" class="0">
 <segment>
 <pinref part="U$1" gate="G$1" pin="VDD"/>
